Commit message: Changed inertia of additional suspension elements to 0

File: rover_simulation/xacro/rocker-bogie/bogie/bogie_link1.xacro (robot description, xacro)
@@ -39,6 +39,6 @@
             <inertial>
                  <origin rpy="0 0 0" xyz="${bogie_link1_offset_x} ${bogie_link1_offset_y*side} ${bogie_link1_offset_z}" />
-                 <mass value="2"/>
-                 <inertia ixx=".003" ixy="0.000" ixz="0.000" iyy=".003" iyz="0.000" izz=".003"/>
+                 <mass value="0"/>
+                 <inertia ixx="0" ixy="0" ixz="0" iyy="0" iyz="0" izz="0"/>
             </inertial>
         </link>

File: rover_simulation/xacro/rocker-bogie/bogie/bogie_link2.xacro (robot description, xacro)
@@ -39,6 +39,6 @@
             <inertial>
                  <origin rpy="0 0 0" xyz="${bogie_link2_offset_x} ${bogie_link2_offset_y*side} ${bogie_link2_offset_z}" />
-                 <mass value="2"/>
-                 <inertia ixx=".003" ixy="0.000" ixz="0.000" iyy=".003" iyz="0.000" izz=".003"/>
+                 <mass value="0"/>
+                 <inertia ixx="0" ixy="0" ixz="0" iyy="0" iyz="0" izz="0"/>
             </inertial>
         </link>

File: rover_simulation/xacro/rocker-bogie/rocker/rocker_link1.xacro (robot description, xacro)
@@ -52,6 +52,6 @@
             <inertial>
                  <origin rpy="0 0 0" xyz="${rocker_link1_offset_x} ${rocker_link1_offset_y} ${rocker_link1_offset_z}" />
-                 <mass value="2"/>
-                 <inertia ixx=".003" ixy="0.000" ixz="0.000" iyy=".003" iyz="0.000" izz=".003"/>
+                 <mass value="0"/>
+                 <inertia ixx="0" ixy="0" ixz="0" iyy="0" iyz="0" izz="0"/>
             </inertial>
         </link>

File: rover_simulation/xacro/rocker-bogie/rocker/rocker_link2.xacro (robot description, xacro)
@@ -26,6 +26,6 @@
             <inertial>
                  <origin rpy="0 0 0" xyz="${rocker_link2_offset_x} ${rocker_link2_offset_y} ${rocker_link2_offset_z}" />
-                 <mass value=".2"/>
-                 <inertia ixx=".003" ixy="0.000" ixz="0.000" iyy=".003" iyz="0.000" izz=".003"/>
+                 <mass value="0"/>
+                 <inertia ixx="0" ixy="0" ixz="0" iyy="0" iyz="0" izz="0"/>
             </inertial>
         </link>

File: rover_simulation/xacro/rocker-bogie/rocker/rocker_link3.xacro (robot description, xacro)
@@ -39,6 +39,6 @@
             <inertial>
                  <origin rpy="0 0 0" xyz="${rocker_link3_offset_x} ${rocker_link3_offset_y} ${rocker_link3_offset_z} " />
-                 <mass value="2"/>
-                 <inertia ixx=".003" ixy="0.000" ixz="0.000" iyy=".003" iyz="0.000" izz=".003"/>
+                 <mass value="0"/>
+                 <inertia ixx="0" ixy="0" ixz="0" iyy="0" iyz="0" izz="0"/>
             </inertial>
         </link>

File: rover_simulation/xacro/rocker-bogie/rocker/rocker_link_diff.xacro (robot description, xacro)
@@ -24,6 +24,6 @@
             </collision>
             <inertial>
-                <mass value=".3"/>
-                <inertia ixx="0.001" ixy="0" ixz="0" iyy="0.001" iyz="0" izz="0.01"/>
+                <mass value="0"/>
+                <inertia ixx="0" ixy="0" ixz="0" iyy="0" iyz="0" izz="0"/>
             </inertial>
         </link>

File: rover_simulation/xacro/rocker-bogie/wheel.xacro (robot description, xacro)
@@ -25,7 +25,7 @@
             </collision>
             <inertial>
-                 <mass value="3"/>
+                 <mass value="1.67"/>
                  <origin xyz="0 0 0" rpy="0 0 0"/>
-                 <inertia ixx=".03" ixy="0.000" ixz="0.000" iyy=".03" iyz="0.000" izz=".03"/>
+                 <inertia ixx=".007228" ixy="0" ixz="0" iyy=".011596" iyz="0" izz=".007228"/>
             </inertial>
         </link>
