Commit message: Added conditional block on __rocker and __bogie bearings inertial, depending on side

File: rover_simulation/xacro/arm/__arm.xacro (robot description, xacro)
@@ -11,5 +11,5 @@
     <xacro:include filename="../sensors/camera.xacro"/>
 <!-- PROPERTIES -->
-    <xacro:property name="manipulator_pose_x" value=".185"/>
+    <xacro:property name="manipulator_pose_x" value=".165"/>
     <xacro:property name="manipulator_pose_z" value=".125"/>
     <xacro:property name="link0_length1" value=".050"/>

File: rover_simulation/xacro/base/main_body.xacro (robot description, xacro)
@@ -8,5 +8,5 @@
         </geometry>
     </xacro:macro>
-    <xacro:macro name="main_body_geometry_2">
+    <!-- <xacro:macro name="main_body_geometry_2">
         <origin rpy="0 0 0" xyz="${body_length/2 + body_translation_x -.125} 0 ${body_height/2 + .050 + body_translation_x}"/>
         <geometry>
@@ -20,5 +20,5 @@
         </geometry>
     </xacro:macro>
-    <xacro:macro name="main_body_geometry_4">                                 <!-- dlugosc przergody - 150 mm -->
+    <xacro:macro name="main_body_geometry_4">
         <origin rpy="0 0 0" xyz="${-body_length/2 + body_translation_x +.025 + 0.100 + 0.150} 0 ${body_height/2 + .050 + body_translation_x}"/>
         <geometry>
@@ -31,5 +31,5 @@
             <box size="${body_length} .050 .100"/>
         </geometry>
-    </xacro:macro>
+    </xacro:macro> -->
 <!-- MATERIAL -->
     <xacro:macro name="main_body_material">
@@ -50,5 +50,5 @@
             </collision>
     <!-- BOXES FOR STONES -->
-            <visual>
+            <!-- <visual>
                 <xacro:main_body_geometry_2/>
                 <xacro:main_body_material/>
@@ -91,5 +91,5 @@
             <collision>
                 <xacro:main_body_geometry_5 side="-1"/>
-            </collision>
+            </collision> -->
             <inertial>
                  <mass value="40"/>
@@ -108,7 +108,4 @@
             <child link="${name}"/>
             <origin rpy="0 0 0" xyz="0 0 0"/>
-            <!--axis xyz="0 1 0"/>
-            <limit effort="100" velocity="1" lower="-.4" upper=".4"/>
-            <dynamics damping="999" friction="999"/-->
         </joint>
         <gazebo reference="${name}_joint">

File: rover_simulation/xacro/rocker-bogie/__rocker-bogie.xacro (robot description, xacro)
@@ -54,6 +54,6 @@
     <xacro:suspension_beam name="suspension_beam"/>
 <!-- SUSPENSION -->
-    <xacro:rocker name="rocker_l" parent="suspension_beam" x="0" y="${suspension_width/2}"    z="0"/>
-    <xacro:rocker name="rocker_r" parent="suspension_beam" x="0" y="${-suspension_width/2}"    z="0"/>
+    <xacro:rocker name="rocker_l" parent="suspension_beam" x="0" y="${suspension_width/2}"    z="0" side="1"/>  <!-- 1 = left -->
+    <xacro:rocker name="rocker_r" parent="suspension_beam" x="0" y="${-suspension_width/2}"    z="0" side="-1"/> <!-- -1 = right -->
     <!-- <xacro:bogie name="bogie_l" parent="rocker_l_bearing" x="${-l_bogie}" y="0"  z="${-h_bogie}" side="1"/>
     <xacro:bogie name="bogie_r" parent="rocker_r_bearing" x="${-l_bogie}" y="0"  z="${-h_bogie}" side="-1"/> -->

File: rover_simulation/xacro/rocker-bogie/bogie/__bogie.xacro (robot description, xacro)
@@ -28,5 +28,5 @@
 <!-- LINKS -->
     <xacro:macro name="bogie" params="name parent x y z side">
-        <xacro:bogie_bearing name="${name}_bearing" parent="${parent}" x="${x}" y="${y}" z="${z}"/>
+        <xacro:bogie_bearing name="${name}_bearing" parent="${parent}" x="${x}" y="${y}" z="${z}" side="${side}"/>
         <xacro:bogie_link1 name="${name}_link1" parent="${name}_bearing"
             x="${bogie_link1_x}" y="${-bogie_link1_y}"  z="${bogie_link1_z}"

File: rover_simulation/xacro/rocker-bogie/bogie/bogie_bearing.xacro (robot description, xacro)
@@ -15,5 +15,5 @@
     </xacro:macro>
 <!-- LINK -->
-    <xacro:macro name="bogie_bearing" params="name parent x y z">
+    <xacro:macro name="bogie_bearing" params="name parent x y z side">
         <link name="${name}">
             <visual>
@@ -26,6 +26,12 @@
             <inertial>
                 <mass value="3"/>
-                <origin xyz="0 0 0" rpy="0 0 0"/>
-                <inertia ixx="0.005" ixy="0" ixz="0" iyy="0.005" iyz="0" izz="0.005"/>
+                <xacro:if value="${side == 1}"> <!-- LEFT-->
+                    <origin xyz="0 0 0" rpy="0 0 0"/>
+                    <inertia ixx="0.005" ixy="0" ixz="0" iyy="0.005" iyz="0" izz="0.005"/>
+                </xacro:if>
+                <xacro:if value="${side == -1}"> <!-- RIGHT-->
+                    <origin xyz="0 0 0" rpy="0 0 0"/>
+                    <inertia ixx="0.005" ixy="0" ixz="0" iyy="0.005" iyz="0" izz="0.005"/>
+                </xacro:if>
             </inertial>
         </link>

File: rover_simulation/xacro/rocker-bogie/rocker/__rocker.xacro (robot description, xacro)
@@ -41,6 +41,6 @@
     <xacro:property name="link_diff_radius" value=".005"/>
 <!-- LINKS -->
-    <xacro:macro name="rocker" params="name parent x y z">
-        <xacro:rocker_bearing name="${name}_bearing" parent="${parent}" x="${x}" y="${y}" z="${z}"/>
+    <xacro:macro name="rocker" params="name parent x y z side">
+        <xacro:rocker_bearing name="${name}_bearing" parent="${parent}" x="${x}" y="${y}" z="${z}" side="${side}"/>
         <xacro:rocker_link1 name="${name}_link1" parent="${name}_bearing"
             x="${rocker_link1_x}" y="${-rocker_link1_y}"  z="${rocker_link1_z}"
@@ -52,5 +52,4 @@
             x="${rocker_link3_x}" y="${-rocker_link3_y}"  z="${rocker_link3_z}"
             pitch="${-rocker_link3_pitch}"/>
-        <!--xacro:link_diff name="${name}_link_diff" parent="${name}_bearing"  x="0" y="0" z="0"/-->
     </xacro:macro>
 </robot>

File: rover_simulation/xacro/rocker-bogie/rocker/rocker_bearing.xacro (robot description, xacro)
@@ -15,5 +15,5 @@
     </xacro:macro>
 <!-- LINK -->
-    <xacro:macro name="rocker_bearing" params="name parent x y z">
+    <xacro:macro name="rocker_bearing" params="name parent x y z side">
         <link name="${name}">
             <visual>
@@ -26,6 +26,12 @@
             <inertial>
                 <mass value="3"/>
-                <origin xyz="0 0 0" rpy="0 0 0"/>
-                <inertia ixx="0.005" ixy="0" ixz="0" iyy="0.005" iyz="0" izz="0.005"/>
+                <xacro:if value="${side == 1}"> <!-- LEFT-->
+                    <origin xyz="0 0 0" rpy="0 0 0"/>
+                    <inertia ixx="0.005" ixy="0" ixz="0" iyy="0.005" iyz="0" izz="0.005"/>
+                </xacro:if>
+                <xacro:if value="${side == -1}"> <!-- RIGHT-->
+                    <origin xyz="0 0 0" rpy="0 0 0"/>
+                    <inertia ixx="0.005" ixy="0" ixz="0" iyy="0.005" iyz="0" izz="0.005"/>
+                </xacro:if>
             </inertial>
         </link>
@@ -38,9 +44,4 @@
                 <dynamics damping="2" friction="0"/>
             </joint>
-            <!--joint name="${name}_joint" type="fixed">
-                <parent link="${parent}"/>
-                <child link="${name}"/>
-                <origin rpy="0 0 0" xyz="${x} ${y} ${z}"/>
-            </joint-->
             <gazebo reference="${name}">
                 <mu1> .2 </mu1>
@@ -49,14 +50,4 @@
                 <selfCollide> True </selfCollide>
             </gazebo>
-            <!--transmission name="${name}_transmission">
-                <type>transmission_interface/SimpleTransmission</type>
-                <joint name="${name}_joint">
-                    <hardwareInterface>EffortJointInterface</hardwareInterface>
-                </joint>
-                <actuator name="${name}_motor">
-                    <hardwareInterface>EffortJointInterface</hardwareInterface>
-                    <mechanicalReduction>1</mechanicalReduction>
-                </actuator>
-            </transmission-->
     </xacro:macro>
 </robot>
