Commit message: Changed link3 limits and reduced link4 mass

File: rover_simulation/xacro/arm/link3.xacro (robot description, xacro)
@@ -41,5 +41,5 @@
             <origin rpy="0 0 0" xyz="${x} ${y} ${z}"/>
             <axis xyz="0 -1 0"/>
-            <limit effort="30" velocity="1" lower="-1.1" upper="2.3"/>
+            <limit effort="30" velocity="1" lower="-2.3" upper="1.1"/>
             <dynamics damping="1"/>
         </joint>

File: rover_simulation/xacro/arm/link4.xacro (robot description, xacro)
@@ -26,5 +26,5 @@
             <inertial>
                 <origin rpy="0 0 0" xyz="${link4_length/2} 0 ${link4_height/2}" />
-                <mass value="1.5"/>
+                <mass value="0.7"/>
                 <inertia ixx=".003" ixy="0.000" ixz="0.000" iyy=".003" iyz="0.000" izz=".003"/>
             </inertial>
