Commit message: Resized suspension and base2

File: rover_simulation/xacro/base/main_body.xacro (robot description, xacro)
@@ -93,6 +93,6 @@
             </collision>
             <inertial>
+                 <mass value="40"/>
                  <origin rpy="0 0 0" xyz="0 0 -.2"/>
-                 <mass value="40"/>
                  <inertia ixx=".1" ixy="0.001" ixz="0.001" iyy=".1" iyz="0.001" izz=".1"/>
             </inertial>

File: rover_simulation/xacro/rocker-bogie/bogie/bogie_bearing.xacro (robot description, xacro)
@@ -26,4 +26,5 @@
             <inertial>
                 <mass value="3"/>
+                <origin xyz="0 0 0" rpy="0 0 0"/>
                 <inertia ixx="0.005" ixy="0" ixz="0" iyy="0.005" iyz="0" izz="0.005"/>
             </inertial>

File: rover_simulation/xacro/rocker-bogie/rocker/rocker_bearing.xacro (robot description, xacro)
@@ -26,4 +26,5 @@
             <inertial>
                 <mass value="3"/>
+                <origin xyz="0 0 0" rpy="0 0 0"/>
                 <inertia ixx="0.005" ixy="0" ixz="0" iyy="0.005" iyz="0" izz="0.005"/>
             </inertial>

File: rover_simulation/xacro/rocker-bogie/wheel.xacro (robot description, xacro)
@@ -26,4 +26,5 @@
             <inertial>
                  <mass value="3"/>
+                 <origin xyz="0 0 0" rpy="0 0 0"/>
                  <inertia ixx=".03" ixy="0.000" ixz="0.000" iyy=".03" iyz="0.000" izz=".03"/>
             </inertial>

Commit message: Inertial of wheel, rocker, bogie and base from Solid model

File: rover_simulation/xacro/base/main_body.xacro (robot description, xacro)
@@ -93,7 +93,7 @@
             </collision> -->
             <inertial>
-                 <mass value="40"/>
-                 <origin rpy="0 0 0" xyz="0 0 -.2"/>
-                 <inertia ixx=".1" ixy="0.001" ixz="0.001" iyy=".1" iyz="0.001" izz=".1"/>
+                 <mass value="16.958705"/>
+                 <origin xyz="-0.151662 0.000004 -0.014131" rpy="0 0 0"/>
+                 <inertia ixx="0.334161" ixy="-0.000002" ixz="0.010911" iyy="0.341848" iyz="0.000000" izz="0.436339"/>
             </inertial>
         </link>

File: rover_simulation/xacro/rocker-bogie/__rocker-bogie.xacro (robot description, xacro)
@@ -6,6 +6,4 @@
     <xacro:include filename="suspension_beam.xacro"/>
     <xacro:include filename="wheel.xacro"/>
-    <!-- TODO NO SUPPORT FOR CLOSED CHAINSD UNTIL URDF 2.0 TODO -->
-    <!--xacro:include filename="rocker-bogie/differential.xacro"/-->
 <!-- PROPERIES -->
     <!-- SUSPENSION PROPERTIES-->
@@ -27,10 +25,6 @@
     <xacro:property name="wheel_base_m" value=".600"/>
     <xacro:property name="wheel_base_b" value=".500"/>
-    <!--xacro:property name="h_bogie" value=".100"/-->
-    <!--xacro:property name="l_bogie" value=".305"/-->
     <xacro:property name="h_wheel" value=".250"/>
     <xacro:property name="l_wheel_f" value=".305"/>
-    <!--xacro:property name="l_wheel_m" value=".160"/>
-    <xacro:property name="l_wheel_b" value=".160"/-->
     <!-- CUSTOM SIM PROPS -->
     <xacro:property name="h_bogie" value=".170"/>
@@ -41,5 +35,5 @@
     <xacro:property name="suspension_beam_length" value=".600"/>
     <xacro:property name="suspension_beam_radius" value=".025"/>
-    <xacro:property name="rocker_bearing_length" value=".050"/>
+    <xacro:property name="rocker_bearing_length" value=".100"/>
     <xacro:property name="rocker_bearing_radius" value=".035"/>
     <xacro:property name="bogie_bearing_length" value=".100"/>
@@ -56,6 +50,4 @@
     <xacro:rocker name="rocker_l" parent="suspension_beam" x="0" y="${suspension_width/2}"    z="0" side="1"/>  <!-- 1 = left -->
     <xacro:rocker name="rocker_r" parent="suspension_beam" x="0" y="${-suspension_width/2}"    z="0" side="-1"/> <!-- -1 = right -->
-    <!-- <xacro:bogie name="bogie_l" parent="rocker_l_bearing" x="${-l_bogie}" y="0"  z="${-h_bogie}" side="1"/>
-    <xacro:bogie name="bogie_r" parent="rocker_r_bearing" x="${-l_bogie}" y="0"  z="${-h_bogie}" side="-1"/> -->
     <xacro:bogie name="bogie_l" parent="rocker_l_bearing" x="${bogie_x}" y="${bogie_y}"  z="${bogie_z}" side="1"/>
     <xacro:bogie name="bogie_r" parent="rocker_r_bearing" x="${bogie_x}" y="${bogie_y}"  z="${bogie_z}" side="-1"/>
@@ -68,10 +60,4 @@
     <xacro:wheel name="br" parent="bogie_r_bearing"  x="${wheel_b_x}" y="${-wheel_b_y}"  z="${wheel_b_z}" u="1"/>
 <!-- MY DIFFERENTIAL PLUGIN -->
-    <!--gazebo>
-        <plugin name="differential" filename="libDifferential.so">
-            <leftJoint>rocker_l_bearing_joint</leftJoint>
-            <rightJoint>rocker_r_bearing_joint</rightJoint>
-        </plugin>
-    </gazebo-->
     <gazebo>
         <plugin name="differential_pid" filename="libDifferentialPID.so">

File: rover_simulation/xacro/rocker-bogie/bogie/__bogie.xacro (robot description, xacro)
@@ -29,10 +29,10 @@
     <xacro:macro name="bogie" params="name parent x y z side">
         <xacro:bogie_bearing name="${name}_bearing" parent="${parent}" x="${x}" y="${y}" z="${z}" side="${side}"/>
-        <xacro:bogie_link1 name="${name}_link1" parent="${name}_bearing"
+        <!-- <xacro:bogie_link1 name="${name}_link1" parent="${name}_bearing"
             x="${bogie_link1_x}" y="${-bogie_link1_y}"  z="${bogie_link1_z}"
             pitch="${-bogie_link1_pitch}" side="${side}"/>
         <xacro:bogie_link2 name="${name}_link2" parent="${name}_bearing"
             x="${bogie_link2_x}" y="${-bogie_link2_y}"  z="${bogie_link2_z}"
-            pitch="${-bogie_link2_pitch}" side="${side}"/>
+            pitch="${-bogie_link2_pitch}" side="${side}"/> -->
     </xacro:macro>
 </robot>

File: rover_simulation/xacro/rocker-bogie/bogie/bogie_bearing.xacro (robot description, xacro)
@@ -25,12 +25,12 @@
             </collision>
             <inertial>
-                <mass value="3"/>
+                <mass value="6.143721"/>
                 <xacro:if value="${side == 1}"> <!-- LEFT-->
-                    <origin xyz="0 0 0" rpy="0 0 0"/>
-                    <inertia ixx="0.005" ixy="0" ixz="0" iyy="0.005" iyz="0" izz="0.005"/>
+                    <origin xyz="-0.000010 0.045682 0.012347" rpy="0 0 0"/>
+                    <inertia ixx="0.082737" ixy="0.015401" ixz="-0.000002" iyy="0.236740" iyz="0.013790" izz="0.176983"/>
                 </xacro:if>
                 <xacro:if value="${side == -1}"> <!-- RIGHT-->
-                    <origin xyz="0 0 0" rpy="0 0 0"/>
-                    <inertia ixx="0.005" ixy="0" ixz="0" iyy="0.005" iyz="0" izz="0.005"/>
+                    <origin xyz="-0.000007 -0.045682 0.012347" rpy="0 0 0"/>
+                    <inertia ixx="0.082737" ixy="-0.015402" ixz="0.000003" iyy="0.236740" iyz="-0.013790" izz="0.176983"/>
                 </xacro:if>
             </inertial>

File: rover_simulation/xacro/rocker-bogie/rocker/__rocker.xacro (robot description, xacro)
@@ -43,5 +43,5 @@
     <xacro:macro name="rocker" params="name parent x y z side">
         <xacro:rocker_bearing name="${name}_bearing" parent="${parent}" x="${x}" y="${y}" z="${z}" side="${side}"/>
-        <xacro:rocker_link1 name="${name}_link1" parent="${name}_bearing"
+        <!-- <xacro:rocker_link1 name="${name}_link1" parent="${name}_bearing"
             x="${rocker_link1_x}" y="${-rocker_link1_y}"  z="${rocker_link1_z}"
             pitch="${-rocker_link1_pitch}"/>
@@ -51,5 +51,5 @@
         <xacro:rocker_link3 name="${name}_link3" parent="${name}_link1"
             x="${rocker_link3_x}" y="${-rocker_link3_y}"  z="${rocker_link3_z}"
-            pitch="${-rocker_link3_pitch}"/>
+            pitch="${-rocker_link3_pitch}"/> -->
     </xacro:macro>
 </robot>

File: rover_simulation/xacro/rocker-bogie/rocker/rocker_bearing.xacro (robot description, xacro)
@@ -27,10 +27,10 @@
                 <mass value="3"/>
                 <xacro:if value="${side == 1}"> <!-- LEFT-->
-                    <origin xyz="0 0 0" rpy="0 0 0"/>
-                    <inertia ixx="0.005" ixy="0" ixz="0" iyy="0.005" iyz="0" izz="0.005"/>
+                    <origin xyz="0.247725 0.035298 -0.066751" rpy="0 0 0"/>
+                    <inertia ixx="0.050813" ixy="0.009439" ixz="-0.021963" iyy="0.135830" iyz="0.004023" izz="0.097893"/>
                 </xacro:if>
                 <xacro:if value="${side == -1}"> <!-- RIGHT-->
-                    <origin xyz="0 0 0" rpy="0 0 0"/>
-                    <inertia ixx="0.005" ixy="0" ixz="0" iyy="0.005" iyz="0" izz="0.005"/>
+                    <origin xyz="0.247727 -0.035298 -0.066751" rpy="0 0 0"/>
+                    <inertia ixx="0.050813" ixy="-0.009439" ixz="-0.021960" iyy="0.135831" iyz="-0.004023" izz="0.097894"/>
                 </xacro:if>
             </inertial>
