Commit message: Resized suspension and base

File: rover_simulation/xacro/base/__base.xacro (robot description, xacro)
@@ -7,9 +7,12 @@
     <xacro:include filename="../sensors/camera.xacro"/>
 <!-- PROPERTIES -->
-    <xacro:property name="body_length" value=".720"/>
+    <!-- <xacro:property name="body_length" value=".720"/>
     <xacro:property name="body_width" value=".400"/>
-    <xacro:property name="body_height" value=".150"/>
-    <xacro:property name="body_translation_x" value="-.080"/>
-    <xacro:property name="body_translation_z" value="-.040"/>
+    <xacro:property name="body_height" value=".150"/> -->
+    <xacro:property name="body_length" value=".570"/>
+    <xacro:property name="body_width" value=".400"/>
+    <xacro:property name="body_height" value=".250"/>
+    <xacro:property name="body_translation_x" value="-.040"/>
+    <xacro:property name="body_translation_z" value="-.0325"/>
     <xacro:property name="tower_pose_x" value="${-body_length/2 - +0.05}"/>
     <xacro:property name="tower_pose_y" value=".160"/>

File: rover_simulation/xacro/rocker-bogie/__rocker-bogie.xacro (robot description, xacro)
@@ -9,4 +9,18 @@
     <!--xacro:include filename="rocker-bogie/differential.xacro"/-->
 <!-- PROPERIES -->
+    <!-- SUSPENSION PROPERTIES-->
+    <xacro:property name="suspension_width" value=".580"/>
+    <xacro:property name="bogie_x" value="-.292"/>
+    <xacro:property name="bogie_y" value=" .000"/>
+    <xacro:property name="bogie_z" value="-.100"/>
+    <xacro:property name="wheel_f_x" value=" .319"/>
+    <xacro:property name="wheel_f_y" value=" .000"/>
+    <xacro:property name="wheel_f_z" value="-.305"/>
+    <xacro:property name="wheel_m_x" value=" .165"/>
+    <xacro:property name="wheel_m_y" value=" .020"/>
+    <xacro:property name="wheel_m_z" value="-.205"/>
+    <xacro:property name="wheel_b_x" value="-.165"/>
+    <xacro:property name="wheel_b_y" value="0"/>
+    <xacro:property name="wheel_b_z" value="-.205"/>
     <!-- WHEELS POSITIONS -->
     <xacro:property name="wheel_base_f" value=".550"/>
@@ -40,15 +54,17 @@
     <xacro:suspension_beam name="suspension_beam"/>
 <!-- SUSPENSION -->
-    <xacro:rocker name="rocker_l" parent="suspension_beam" x="0" y="${wheel_base_m/2}"    z="0"/>
-    <xacro:rocker name="rocker_r" parent="suspension_beam" x="0" y="${-wheel_base_m/2}"    z="0"/>
-    <xacro:bogie name="bogie_l" parent="rocker_l_bearing" x="${-l_bogie}" y="0"  z="${-h_bogie}" side="1"/>
-    <xacro:bogie name="bogie_r" parent="rocker_r_bearing" x="${-l_bogie}" y="0"  z="${-h_bogie}" side="-1"/>
+    <xacro:rocker name="rocker_l" parent="suspension_beam" x="0" y="${suspension_width/2}"    z="0"/>
+    <xacro:rocker name="rocker_r" parent="suspension_beam" x="0" y="${-suspension_width/2}"    z="0"/>
+    <!-- <xacro:bogie name="bogie_l" parent="rocker_l_bearing" x="${-l_bogie}" y="0"  z="${-h_bogie}" side="1"/>
+    <xacro:bogie name="bogie_r" parent="rocker_r_bearing" x="${-l_bogie}" y="0"  z="${-h_bogie}" side="-1"/> -->
+    <xacro:bogie name="bogie_l" parent="rocker_l_bearing" x="${bogie_x}" y="${bogie_y}"  z="${bogie_z}" side="1"/>
+    <xacro:bogie name="bogie_r" parent="rocker_r_bearing" x="${bogie_x}" y="${bogie_y}"  z="${bogie_z}" side="-1"/>
 <!-- WHEELS -->
-    <xacro:wheel name="fl" parent="rocker_l_bearing" x="${l_wheel_f}"    z="${-h_wheel}"    y="${+f_wheel_deviation + wheel_offset}" u="1"/>
-    <xacro:wheel name="fr" parent="rocker_r_bearing" x="${l_wheel_f}"    z="${-h_wheel}"    y="${-f_wheel_deviation - wheel_offset}" u="1"/>
-    <xacro:wheel name="ml" parent="bogie_l_bearing"  x="${l_wheel_m}"    z="${-h_wheel+h_bogie}"    y="${+wheel_offset}" u=".7"/>
-    <xacro:wheel name="mr" parent="bogie_r_bearing"  x="${l_wheel_m}"    z="${-h_wheel+h_bogie}"    y="${-wheel_offset}" u=".7"/>
-    <xacro:wheel name="bl" parent="bogie_l_bearing"  x="${-l_wheel_b}"   z="${-h_wheel+h_bogie}"    y="${+b_wheel_deviation + wheel_offset}" u="1"/>
-    <xacro:wheel name="br" parent="bogie_r_bearing"  x="${-l_wheel_b}"   z="${-h_wheel+h_bogie}"    y="${-b_wheel_deviation - wheel_offset}" u="1"/>
+    <xacro:wheel name="fl" parent="rocker_l_bearing" x="${wheel_f_x}" y="${+wheel_f_y}"  z="${wheel_f_z}" u="1"/>
+    <xacro:wheel name="fr" parent="rocker_r_bearing" x="${wheel_f_x}" y="${-wheel_f_y}"  z="${wheel_f_z}" u="1"/>
+    <xacro:wheel name="ml" parent="bogie_l_bearing"  x="${wheel_m_x}" y="${+wheel_m_y}"  z="${wheel_m_z}" u=".7"/>
+    <xacro:wheel name="mr" parent="bogie_r_bearing"  x="${wheel_m_x}" y="${-wheel_m_y}"  z="${wheel_m_z}" u=".7"/>
+    <xacro:wheel name="bl" parent="bogie_l_bearing"  x="${wheel_b_x}" y="${+wheel_b_y}"  z="${wheel_b_z}" u="1"/>
+    <xacro:wheel name="br" parent="bogie_r_bearing"  x="${wheel_b_x}" y="${-wheel_b_y}"  z="${wheel_b_z}" u="1"/>
 <!-- MY DIFFERENTIAL PLUGIN -->
     <!--gazebo>

Commit message: PID Tuinig ,wheel orientation(1 contact point for flat surface) and friction change

File: rover_simulation/xacro/base/__base.xacro (robot description, xacro)
@@ -24,13 +24,12 @@
     <xacro:property name="tower_pitch_height" value=".050"/>
 <!-- BODY -->
-    <!--xacro:main_body name="main_body" parent="rocker_l_bearing" x="${body_translation_x}" z="${wheel_base_m/2}" y="${body_translation_z}"/-->
     <xacro:main_body name="main_body" parent="suspension_beam" x="${body_translation_x}" y="0" z="${body_translation_z}"/>
 <!--TOWER -->
-    <xacro:tower_yaw name="tower_yaw" parent="main_body" x="${tower_pose_x}" y="${tower_pose_y}" z="${tower_pose_z}"/>
-    <xacro:tower_pitch name="tower_pitch" parent="tower_yaw" x="0" y="0" z="${tower_yaw_height/2}"/>
+    <!-- <xacro:tower_yaw name="tower_yaw" parent="main_body" x="${tower_pose_x}" y="${tower_pose_y}" z="${tower_pose_z}"/>
+    <xacro:tower_pitch name="tower_pitch" parent="tower_yaw" x="0" y="0" z="${tower_yaw_height/2}"/> -->
 <!-- SENSORS -->
     <xacro:camera_link name="camera1" parent="main_body" x="${body_length/2 + camera_x/2 + body_translation_x}" y=".100" z="-.070" pitch="0"/>
     <xacro:camera_link name="camera2" parent="main_body" x="${body_length/2 + camera_x/2 + body_translation_x}" y="-.100" z="-.070" pitch="0"/>
-    <xacro:camera_link name="camera3" parent="tower_pitch" x="${tower_pitch_length/2 + camera_x/2}" y="0" z="0" pitch="0"/>
-    <xacro:camera_link name="camera5" parent="main_body" x="0" y="0" z="${-body_height/2 - camera_x/2 + body_translation_z}" pitch="1.57075"/>
+    <!-- <xacro:camera_link name="camera3" parent="tower_pitch" x="${tower_pitch_length/2 + camera_x/2}" y="0" z="0" pitch="0"/> -->
+    <!-- <xacro:camera_link name="camera5" parent="main_body" x="0" y="0" z="${-body_height/2 - camera_x/2 + body_translation_z}" pitch="1.57075"/> -->
 </robot>

File: rover_simulation/xacro/rocker-bogie/__rocker-bogie.xacro (robot description, xacro)
@@ -53,10 +53,10 @@
     <xacro:bogie name="bogie_r" parent="rocker_r_bearing" x="${bogie_x}" y="${bogie_y}"  z="${bogie_z}" side="-1"/>
 <!-- WHEELS -->
-    <xacro:wheel name="fl" parent="rocker_l_bearing" x="${wheel_f_x}" y="${+wheel_f_y}"  z="${wheel_f_z}" u="1"/>
-    <xacro:wheel name="fr" parent="rocker_r_bearing" x="${wheel_f_x}" y="${-wheel_f_y}"  z="${wheel_f_z}" u="1"/>
-    <xacro:wheel name="ml" parent="bogie_l_bearing"  x="${wheel_m_x}" y="${+wheel_m_y}"  z="${wheel_m_z}" u=".7"/>
-    <xacro:wheel name="mr" parent="bogie_r_bearing"  x="${wheel_m_x}" y="${-wheel_m_y}"  z="${wheel_m_z}" u=".7"/>
-    <xacro:wheel name="bl" parent="bogie_l_bearing"  x="${wheel_b_x}" y="${+wheel_b_y}"  z="${wheel_b_z}" u="1"/>
-    <xacro:wheel name="br" parent="bogie_r_bearing"  x="${wheel_b_x}" y="${-wheel_b_y}"  z="${wheel_b_z}" u="1"/>
+    <xacro:wheel name="fl" parent="rocker_l_bearing" x="${wheel_f_x}" y="${+wheel_f_y}"  z="${wheel_f_z}" side="1"/>
+    <xacro:wheel name="fr" parent="rocker_r_bearing" x="${wheel_f_x}" y="${-wheel_f_y}"  z="${wheel_f_z}" side="-1"/>
+    <xacro:wheel name="ml" parent="bogie_l_bearing"  x="${wheel_m_x}" y="${+wheel_m_y}"  z="${wheel_m_z}" side="1"/>
+    <xacro:wheel name="mr" parent="bogie_r_bearing"  x="${wheel_m_x}" y="${-wheel_m_y}"  z="${wheel_m_z}" side="-1"/>
+    <xacro:wheel name="bl" parent="bogie_l_bearing"  x="${wheel_b_x}" y="${+wheel_b_y}"  z="${wheel_b_z}" side="1"/>
+    <xacro:wheel name="br" parent="bogie_r_bearing"  x="${wheel_b_x}" y="${-wheel_b_y}"  z="${wheel_b_z}" side="-1"/>
 <!-- MY DIFFERENTIAL PLUGIN -->
     <gazebo>
@@ -65,7 +65,7 @@
             <rightJoint>rocker_r_bearing_joint</rightJoint>
             <topic>/rover/differential_pid</topic>
-            <Kp>3000</Kp>
+            <Kp>1000</Kp>
             <Ki>0</Ki>
-            <Kd>10000</Kd>
+            <Kd>3000</Kd>
             <limit>10000</limit>
         </plugin>

File: rover_simulation/xacro/rocker-bogie/wheel.xacro (robot description, xacro)
@@ -15,5 +15,5 @@
     </xacro:macro>
 <!-- LINK -->
-    <xacro:macro name="wheel" params="name parent x y z u">
+    <xacro:macro name="wheel" params="name parent x y z side">
         <link name="wheel_${name}">
             <visual>
@@ -33,5 +33,5 @@
             <parent link="${parent}"/>
             <child link="wheel_${name}"/>
-            <origin rpy="0 0 0" xyz="${x} ${y} ${z}"/>
+            <origin rpy="${-side*0.02} 0 0" xyz="${x} ${y} ${z}"/>
             <axis xyz="0 1 0"/>
             <limit effort="100" velocity="10"/>
@@ -39,9 +39,11 @@
         </joint>
         <gazebo reference="wheel_${name}">
-            <mu1> ${u} </mu1>
-            <mu2> ${u} </mu2>
-            <!--fdir1> 0 1 0 </fdir1-->
-            <material> Gazebo/Black </material>
-            <selfCollide> True </selfCollide>
+            <mu1 value="0.5"/>
+            <mu2 value="0.5"/>
+            <!-- <kp  value="10000000.0" /> -->
+            <!-- <kd  value="1.0" /> -->
+            <!-- <fdir1 value="0 1 0"/> -->
+            <material value="Gazebo/Black"/>
+            <selfCollide value="True"/>
         </gazebo>
         <gazebo>
@@ -57,7 +59,7 @@
                 <joint>wheel_${name}_joint</joint>
                 <topic>/rover/wheel_${name}_velocity_controller</topic>
-                <Kp>5</Kp>
-                <Ki>0.5</Ki>
-                <Kd>0.4</Kd>
+                <Kp>2</Kp>
+                <Ki>0.1</Ki>
+                <Kd>0.1</Kd>
                 <limit>100</limit>
             </plugin>

File: rover_simulation/xacro/rover.xacro (robot description, xacro)
@@ -8,4 +8,4 @@
     <xacro:include filename="rocker-bogie/__rocker-bogie.xacro"/>
     <xacro:include filename="base/__base.xacro"/>
-    <xacro:include filename="arm/__arm.xacro"/>
+    <!-- <xacro:include filename="arm/__arm.xacro"/> -->
 </robot>
