Commit message: Working dynamometer, changed plugin location in .xacro

File: rover_simulation/xacro/rocker-bogie/__rocker-bogie.xacro (robot description, xacro)
@@ -71,3 +71,16 @@
         </plugin>
     </gazebo>
+ <!-- DYNAMOMETER PLUGINS -->
+    <gazebo>
+        <plugin name="rocker_l_bearing_joint_dynamometer" filename="libJointDynamometer.so">
+            <joint>rocker_l_bearing_joint</joint>
+            <topic>/rover/joint_dynamometer/rocker_l_bearing_joint</topic>
+        </plugin>
+    </gazebo>
+    <gazebo>
+        <plugin name="rocker_r_bearing_joint_dynamometer" filename="libJointDynamometer.so">
+            <joint>rocker_r_bearing_joint</joint>
+            <topic>/rover/joint_dynamometer/rocker_r_bearing_joint</topic>
+        </plugin>
+    </gazebo>
 </robot>

File: rover_simulation/xacro/rocker-bogie/rocker/rocker_bearing.xacro (robot description, xacro)
@@ -36,4 +36,10 @@
             </inertial>
         </link>
+        <gazebo reference="${name}">
+            <mu1> .2 </mu1>
+            <mu2> .2 </mu2>
+            <material> Gazebo/Grey </material>
+            <selfCollide> True </selfCollide>
+        </gazebo>
             <joint name="${name}_joint" type="revolute">
                 <parent link="${parent}"/>
@@ -44,9 +50,6 @@
                 <dynamics damping="2" friction="0"/>
             </joint>
-            <gazebo reference="${name}">
-                <mu1> .2 </mu1>
-                <mu2> .2 </mu2>
-                <material> Gazebo/Grey </material>
-                <selfCollide> True </selfCollide>
+            <gazebo reference="${name}_joint">
+                <provideFeedback value="true"/>
             </gazebo>
     </xacro:macro>

File: rover_simulation/xacro/rocker-bogie/suspension_beam.xacro (robot description, xacro)
@@ -33,6 +33,6 @@
             </collision>
             <inertial>
-                <mass value="3"/>
-                <inertia ixx="0.005" ixy="0" ixz="0" iyy="0.005" iyz="0" izz="0.005"/>
+                <mass value="0.001"/>
+                <inertia ixx="0.000005" ixy="0" ixz="0" iyy="0.000005" iyz="0" izz="0.000005"/>
             </inertial>
         </link>

File: rover_simulation/xacro/sensors/camera.xacro (robot description, xacro)
@@ -84,5 +84,5 @@
             <inertial>
                  <mass value=".01"/>
-                 <inertia ixx=".003" ixy="0" ixz="0" iyy=".003" iyz="0" izz=".003"/>
+                 <inertia ixx=".00000003" ixy="0" ixz="0" iyy=".00000003" iyz="0" izz=".00000003"/>
             </inertial>
         </link>

Commit message: joint_dynamometer: file opend and closed with each write model: added joint dynamometer to wheels and bogie bearing

File: rover_simulation/xacro/rocker-bogie/__rocker-bogie.xacro (robot description, xacro)
@@ -84,3 +84,51 @@
         </plugin>
     </gazebo>
+    <gazebo>
+        <plugin name="bogie_l_bearing_joint_dynamometer" filename="libJointDynamometer.so">
+            <joint>bogie_l_bearing_joint</joint>
+            <topic>/rover/joint_dynamometer/bogie_l_bearing_joint</topic>
+        </plugin>
+    </gazebo>
+    <gazebo>
+        <plugin name="bogie_r_bearing_joint_dynamometer" filename="libJointDynamometer.so">
+            <joint>bogie_r_bearing_joint</joint>
+            <topic>/rover/joint_dynamometer/bogie_r_bearing_joint</topic>
+        </plugin>
+    </gazebo>
+    <gazebo>
+        <plugin name="wheel_fl_joint_dynamometer" filename="libJointDynamometer.so">
+            <joint>wheel_fl_joint</joint>
+            <topic>/rover/joint_dynamometer/wheel_fl_joint</topic>
+        </plugin>
+    </gazebo>
+    <gazebo>
+        <plugin name="wheel_fr_joint_dynamometer" filename="libJointDynamometer.so">
+            <joint>wheel_fr_joint</joint>
+            <topic>/rover/joint_dynamometer/wheel_fr_joint</topic>
+        </plugin>
+    </gazebo>
+    <gazebo>
+        <plugin name="wheel_ml_joint_dynamometer" filename="libJointDynamometer.so">
+            <joint>wheel_ml_joint</joint>
+            <topic>/rover/joint_dynamometer/wheel_ml_joint</topic>
+        </plugin>
+    </gazebo>
+    <gazebo>
+        <plugin name="wheel_mr_joint_dynamometer" filename="libJointDynamometer.so">
+            <joint>wheel_mr_joint</joint>
+            <topic>/rover/joint_dynamometer/wheel_mr_joint</topic>
+        </plugin>
+    </gazebo>
+    <gazebo>
+        <plugin name="wheel_bl_joint_dynamometer" filename="libJointDynamometer.so">
+            <joint>wheel_bl_joint</joint>
+            <topic>/rover/joint_dynamometer/wheel_bl_joint</topic>
+        </plugin>
+    </gazebo>
+    <gazebo>
+        <plugin name="wheel_br_joint_dynamometer" filename="libJointDynamometer.so">
+            <joint>wheel_br_joint</joint>
+            <topic>/rover/joint_dynamometer/wheel_br_joint</topic>
+        </plugin>
+    </gazebo>
 </robot>

File: rover_simulation/xacro/rocker-bogie/bogie/bogie_bearing.xacro (robot description, xacro)
@@ -36,4 +36,10 @@
             </inertial>
         </link>
+        <gazebo reference="${name}">
+            <mu1> .2 </mu1>
+            <mu2> .2 </mu2>
+            <material> Gazebo/Grey </material>
+            <selfCollide> True </selfCollide>
+        </gazebo>
             <joint name="${name}_joint" type="revolute">
                 <parent link="${parent}"/>
@@ -44,9 +50,6 @@
                 <dynamics damping="1"/>
             </joint>
-            <gazebo reference="${name}">
-                <mu1> .2 </mu1>
-                <mu2> .2 </mu2>
-                <material> Gazebo/Grey </material>
-                <selfCollide> True </selfCollide>
+            <gazebo reference="${name}_joint">
+                <provideFeedback value="true"/>
             </gazebo>
             <transmission name="${name}_transmission">

File: rover_simulation/xacro/rocker-bogie/wheel.xacro (robot description, xacro)
@@ -30,4 +30,13 @@
             </inertial>
         </link>
+        <gazebo reference="wheel_${name}">
+            <mu1 value="0.5"/>
+            <mu2 value="0.5"/>
+            <!-- <kp  value="10000.0" /> -->
+            <!-- <kd  value="10000.0" /> -->
+            <!-- <fdir1 value="0 1 0"/> -->
+            <material value="Gazebo/Black"/>
+            <selfCollide value="True"/>
+        </gazebo>
         <joint name="wheel_${name}_joint" type="continuous">
             <parent link="${parent}"/>
@@ -38,12 +47,6 @@
             <dynamics damping="1"/>
         </joint>
-        <gazebo reference="wheel_${name}">
-            <mu1 value="0.5"/>
-            <mu2 value="0.5"/>
-            <!-- <kp  value="10000.0" /> -->
-            <!-- <kd  value="10000.0" /> -->
-            <!-- <fdir1 value="0 1 0"/> -->
-            <material value="Gazebo/Black"/>
-            <selfCollide value="True"/>
+        <gazebo reference="wheel_${name}_joint">
+            <provideFeedback value="true"/>
         </gazebo>
         <gazebo>
