Commit message: add uart_433_simulation_bridge

File: phobos_simulation/xacro/arm/finger.xacro (robot description, xacro)
@@ -91,7 +91,7 @@
         </gazebo-->
         <gazebo>
-            <plugin name="${name}_joint_limiter" filename="libJointLimiter.so">
+            <plugin name="joint_limiter_${name}" filename="libJointLimiter.so">
                 <joint>${name}_joint</joint>
-                <topic>/rover/${name}_velocity_controller</topic>
+                <topic>/simulation/controller/vel/${name}</topic>
                 <lower>0</lower>
                 <upper>${link4_width/2 - finger_width}</upper>
@@ -99,7 +99,7 @@
         </gazebo>
         <gazebo>
-            <plugin name="${name}_controller" filename="libControllerPID.so">
+            <plugin name="joint_controller${name}" filename="libControllerPID.so">
                 <joint>${name}_joint</joint>
-                <topic>/rover/${name}_velocity_controller</topic>
+                <topic>/simulation/controller/vel/${name}</topic>
                 <Kp>10</Kp>
                 <Ki>0</Ki>

File: phobos_simulation/xacro/arm/finger_b.xacro (robot description, xacro)
@@ -88,7 +88,7 @@
         </gazebo-->
         <!--gazebo>
-            <plugin name="${name}_joint_limiter" filename="libJointLimiter.so">
+            <plugin name="joint_limiter_${name}" filename="libJointLimiter.so">
                 <joint>${name}_joint</joint>
-                <topic>/rover/${name}_velocity_controller</topic>
+                <topic>/simulation/controller/vel/${name}</topic>
                 <lower>0</lower>
                 <upper>${link4_width/2 - finger_b_width}</upper>
@@ -96,7 +96,7 @@
         </gazebo>
         <gazebo>
-            <plugin name="${name}_controller" filename="libControllerPID.so">
+            <plugin name="joint_controller_${name}" filename="libControllerPID.so">
                 <joint>${name}_joint</joint>
-                <topic>/rover/${name}_velocity_controller</topic>
+                <topic>/simulation/controller/vel/${name}</topic>
                 <Kp>10</Kp>
                 <Ki>0</Ki>

File: phobos_simulation/xacro/arm/link0.xacro (robot description, xacro)
@@ -68,7 +68,7 @@
         </gazebo-->
         <gazebo>
-            <plugin name="${name}_joint_limiter" filename="libJointLimiter.so">
+            <plugin name="joint_limiter_${name}" filename="libJointLimiter.so">
                 <joint>${name}_joint</joint>
-                <topic>/rover/${name}_velocity_controller</topic>
+                <topic>/simulation/controller/vel/${name}</topic>
                 <lower>-3</lower>
                 <upper>3</upper>
@@ -76,7 +76,17 @@
         </gazebo>
         <gazebo>
-            <plugin name="${name}_controller" filename="libControllerPID.so">
+            <plugin name="joint_encoder_${name}" filename="libJointEncoder.so">
                 <joint>${name}_joint</joint>
-                <topic>/rover/${name}_velocity_controller</topic>
+                <topic>/simulation/encoder/abs/${name}</topic>
+                <lower>-3</lower>
+                <upper>3</upper>
+                <absolute>1</absolute>
+                <resolution>3600</resolution>
+            </plugin>
+        </gazebo>
+        <gazebo>
+            <plugin name="joint_controller_${name}" filename="libControllerPID.so">
+                <joint>${name}_joint</joint>
+                <topic>/simulation/controller/vel/${name}</topic>
                 <Kp>20</Kp>
                 <Ki>2</Ki>

File: phobos_simulation/xacro/arm/link1.xacro (robot description, xacro)
@@ -65,7 +65,7 @@
         </gazebo-->
         <gazebo>
-            <plugin name="${name}_joint_limiter" filename="libJointLimiter.so">
+            <plugin name="joint_limiter_${name}" filename="libJointLimiter.so">
                 <joint>${name}_joint</joint>
-                <topic>/rover/${name}_velocity_controller</topic>
+                <topic>/simulation/controller/vel/${name}</topic>
                 <lower>-1.25</lower>
                 <upper>1.6</upper>
@@ -73,7 +73,17 @@
         </gazebo>
         <gazebo>
-            <plugin name="${name}_controller" filename="libControllerPID.so">
+            <plugin name="joint_encoder_${name}" filename="libJointEncoder.so">
                 <joint>${name}_joint</joint>
-                <topic>/rover/${name}_velocity_controller</topic>
+                <topic>/simulation/encoder/abs/${name}</topic>
+                <lower>-1.25</lower>
+                <upper>1.6</upper>
+                <absolute>1</absolute>
+                <resolution>3600</resolution>
+            </plugin>
+        </gazebo>
+        <gazebo>
+            <plugin name="joint_controller_${name}" filename="libControllerPID.so">
+                <joint>${name}_joint</joint>
+                <topic>/simulation/controller/vel/${name}</topic>
                 <Kp>30</Kp>
                 <Ki>3</Ki>

File: phobos_simulation/xacro/arm/link2.xacro (robot description, xacro)
@@ -65,7 +65,7 @@
         </gazebo-->
         <gazebo>
-            <plugin name="${name}_joint_limiter" filename="libJointLimiter.so">
+            <plugin name="joint_limiter_${name}" filename="libJointLimiter.so">
                 <joint>${name}_joint</joint>
-                <topic>/rover/${name}_velocity_controller</topic>
+                <topic>/simulation/controller/vel/${name}</topic>
                 <lower>0</lower>
                 <upper>3.65</upper>
@@ -73,7 +73,17 @@
         </gazebo>
         <gazebo>
-            <plugin name="${name}_controller" filename="libControllerPID.so">
+            <plugin name="joint_encoder_${name}" filename="libJointEncoder.so">
                 <joint>${name}_joint</joint>
-                <topic>/rover/${name}_velocity_controller</topic>
+                <topic>/simulation/encoder/abs/${name}</topic>
+                <lower>0</lower>
+                <upper>3.65</upper>
+                <absolute>1</absolute>
+                <resolution>3600</resolution>
+            </plugin>
+        </gazebo>
+        <gazebo>
+            <plugin name="joint_controller_${name}" filename="libControllerPID.so">
+                <joint>${name}_joint</joint>
+                <topic>/simulation/controller/vel/${name}</topic>
                 <Kp>30</Kp>
                 <Ki>3</Ki>

File: phobos_simulation/xacro/arm/link3.xacro (robot description, xacro)
@@ -52,7 +52,7 @@
         </gazebo-->
         <gazebo>
-            <plugin name="${name}_joint_limiter" filename="libJointLimiter.so">
+            <plugin name="joint_limiter_${name}" filename="libJointLimiter.so">
                 <joint>${name}_joint</joint>
-                <topic>/rover/${name}_velocity_controller</topic>
+                <topic>/simulation/controller/vel/${name}</topic>
                 <lower>-2.3</lower>
                 <upper>1.1</upper>
@@ -60,7 +60,17 @@
         </gazebo>
         <gazebo>
-            <plugin name="${name}_controller" filename="libControllerPID.so">
+            <plugin name="joint_encoder_${name}" filename="libJointEncoder.so">
                 <joint>${name}_joint</joint>
-                <topic>/rover/${name}_velocity_controller</topic>
+                <topic>/simulation/encoder/abs/${name}</topic>
+                <lower>-2.3</lower>
+                <upper>1.1</upper>
+                <absolute>1</absolute>
+                <resolution>3600</resolution>
+            </plugin>
+        </gazebo>
+        <gazebo>
+            <plugin name="joint_controller_${name}" filename="libControllerPID.so">
+                <joint>${name}_joint</joint>
+                <topic>/simulation/controller/vel/${name}</topic>
                 <Kp>20</Kp>
                 <Ki>0</Ki>

File: phobos_simulation/xacro/arm/link4.xacro (robot description, xacro)
@@ -52,7 +52,7 @@
         </gazebo-->
         <gazebo>
-            <plugin name="${name}_joint_limiter" filename="libJointLimiter.so">
+            <plugin name="joint_limiter_${name}" filename="libJointLimiter.so">
                 <joint>${name}_joint</joint>
-                <topic>/rover/${name}_velocity_controller</topic>
+                <topic>/simulation/controller/vel/${name}</topic>
                 <lower>-3.14</lower>
                 <upper>3.14</upper>
@@ -60,7 +60,17 @@
         </gazebo>
         <gazebo>
-            <plugin name="${name}_controller" filename="libControllerPID.so">
+            <plugin name="joint_encoder_${name}" filename="libJointEncoder.so">
                 <joint>${name}_joint</joint>
-                <topic>/rover/${name}_velocity_controller</topic>
+                <topic>/simulation/encoder/abs/${name}</topic>
+                <lower>-3.14</lower>
+                <upper>3.14</upper>
+                <absolute>1</absolute>
+                <resolution>3600</resolution>
+            </plugin>
+        </gazebo>
+        <gazebo>
+            <plugin name="joint_controller_${name}" filename="libControllerPID.so">
+                <joint>${name}_joint</joint>
+                <topic>/simulation/controller/vel/${name}</topic>
                 <Kp>1.05</Kp>
                 <Ki>0</Ki>

File: phobos_simulation/xacro/base/tower_pitch.xacro (robot description, xacro)
@@ -44,7 +44,7 @@
             </gazebo>
             <gazebo>
-                <plugin name="${name}_joint_limiter" filename="libJointLimiter.so">
+                <plugin name="joint_limiter_${name}" filename="libJointLimiter.so">
                     <joint>${name}_joint</joint>
-                    <topic>/rover/${name}_velocity_controller</topic>
+                    <topic>/simulation/controller/vel/${name}</topic>
                     <lower>-0.785</lower>
                     <upper>0.785</upper>
@@ -52,7 +52,7 @@
             </gazebo>
             <gazebo>
-                <plugin name="${name}_controller" filename="libControllerPID.so">
+                <plugin name="joint_controller_${name}" filename="libControllerPID.so">
                     <joint>${name}_joint</joint>
-                    <topic>/rover/${name}_velocity_controller</topic>
+                    <topic>/simulation/controller/vel/${name}</topic>
                     <Kp>0.8</Kp>
                     <Ki>0.25</Ki>

File: phobos_simulation/xacro/base/tower_yaw.xacro (robot description, xacro)
@@ -41,7 +41,7 @@
             </gazebo>
             <gazebo>
-                <plugin name="${name}_joint_limiter" filename="libJointLimiter.so">
+                <plugin name="joint_limiter_${name}" filename="libJointLimiter.so">
                     <joint>${name}_joint</joint>
-                    <topic>/rover/${name}_velocity_controller</topic>
+                    <topic>/simulation/controller/vel/${name}</topic>
                     <lower>-3.14</lower>
                     <upper>3.14</upper>
@@ -49,7 +49,7 @@
             </gazebo>
             <gazebo>
-                <plugin name="${name}_controller" filename="libControllerPID.so">
+                <plugin name="joint_controller_${name}" filename="libControllerPID.so">
                     <joint>${name}_joint</joint>
-                    <topic>/rover/${name}_velocity_controller</topic>
+                    <topic>/simulation/controller/vel/${name}</topic>
                     <Kp>1</Kp>
                     <Ki>0.7</Ki>

File: phobos_simulation/xacro/rocker-bogie/wheel.xacro (robot description, xacro)
@@ -51,7 +51,7 @@
         </gazebo>
         <gazebo>
-            <plugin name="wheel_${name}_joint_limiter" filename="libJointLimiter.so">
+            <plugin name="joint_limiter_wheel_${name}" filename="libJointLimiter.so">
                 <joint>wheel_${name}_joint</joint>
-                <topic>/rover/wheel_${name}_velocity_controller</topic>
+                <topic>/simulation/controller/vel/wheel_${name}</topic>
                 <lower>-9999999</lower>
                 <upper>9999999</upper>
@@ -59,7 +59,17 @@
         </gazebo>
         <gazebo>
-            <plugin name="wheel_${name}_controller" filename="libControllerPID.so">
+            <plugin name="joint_encoder_wheel_${name}" filename="libJointEncoder.so">
                 <joint>wheel_${name}_joint</joint>
-                <topic>/rover/wheel_${name}_velocity_controller</topic>
+                <topic>/simulation/encoder/rel/wheel_${name}</topic>
+                <lower>0</lower>
+                <upper>9999999</upper>
+                <absolute>0</absolute>
+                <resolution>3600</resolution>
+            </plugin>
+        </gazebo>
+        <gazebo>
+            <plugin name="joint_controller_wheel_${name}" filename="libControllerPID.so">
+                <joint>wheel_${name}_joint</joint>
+                <topic>/simulation/controller/vel/wheel_${name}</topic>
                 <Kp>2</Kp>
                 <Ki>0.1</Ki>
