Commit message: MESHES for manipulators link 0,1,2,3,4

File: phobos_simulation/xacro/arm/link_4.xacro (robot description, xacro)
@@ -10,5 +10,5 @@
     <!-- VISUAL -->
     <xacro:macro name="link_4_visual">
-        <origin xyz="0 0 0" rpy="0.1 0 0"/>
+        <origin xyz="0.25 0.1 -0.587" rpy="1.57075 -0.15 -1.45"/>
         <geometry>
             <mesh filename="package://phobos_meshes/rover_stl/chwytak.STL" scale="0.001 0.001 0.001"/>
