Commit message: All tf's working - finger_l as gripper pose

File: phobos_simulation/xacro/arm/__arm.xacro (robot description, xacro)
@@ -39,9 +39,9 @@
     <xacro:link_4 name="link_4" parent="link_3"    x="${link_3_length}"     y="0"    z="0"/>
 <!-- GRABBER -->
-    <xacro:finger name="finger1" parent="link_4" x="${link_4_length + finger_length/2}" y="${link_4_width/2 - finger_width/2}" z="${finger_height+.001}" side="-1"/>
-    <xacro:finger_b name="finger1b" parent="finger1" x="0" y="0" z="${-2*finger_height-.001}" side="-1"/>
-    <xacro:finger name="finger2" parent="link_4" x="${link_4_length + finger_length/2}" y="${-link_4_width/2 + finger_width/2}" z="0" side="1"/>
-    <xacro:finger_b name="finger2c" parent="finger2" x="0" y="0" z="${2*finger_height+.002}" side="1"/>
-    <xacro:finger_b name="finger2b" parent="finger2" x="0" y="0" z="${-2*finger_height-.002}" side="1"/>
+    <xacro:finger name="finger_l" parent="link_4" x="${link_4_length + finger_length/2}" y="${link_4_width/2 - finger_width/2-.001}" z="${finger_height+.001}" side="-1"/>
+    <xacro:finger_b name="finger_lb" parent="finger_l" x="0" y="0" z="${-2*finger_height-.001}" side="-1"/>
+    <xacro:finger name="finger_r" parent="link_4" x="${link_4_length + finger_length/2}" y="${-link_4_width/2 + finger_width/2}" z="0" side="1"/>
+    <xacro:finger_b name="finger_rc" parent="finger_r" x="0" y="0" z="${2*finger_height+.002}" side="1"/>
+    <xacro:finger_b name="finger_rb" parent="finger_r" x="0" y="0" z="${-2*finger_height-.002}" side="1"/>
 <!-- SENSORS -->
     <xacro:camera_link name="camera4" parent="link_4" x=".030" y="0" z=".100" pitch="0.4"/>

File: phobos_simulation/xacro/arm/finger.xacro (robot description, xacro)
@@ -80,5 +80,5 @@
             <origin rpy="0 0 0" xyz="${x} ${y} ${z}"/>
             <axis xyz="0 ${side*1} 0"/>
-            <limit effort="100" velocity="1" lower="0" upper="${link_4_width/2 - finger_width}"/>
+            <limit effort="10000" velocity="1" lower="0" upper="${link_4_width/2 - finger_width}"/>
             <dynamics damping=".1"/>
         </joint>
@@ -99,9 +99,29 @@
         </gazebo>
         <gazebo>
+            <plugin name="joint_encoder_${name}" filename="libJointEncoder.so">
+                <joint>${name}_joint</joint>
+                <topic>/simulation/encoder/abs/${name}</topic>
+                <lower>0</lower>
+                <upper>${link_4_width/2 - finger_width}</upper>
+                <absolute>1</absolute>
+                <resolution>10000</resolution>
+            </plugin>
+        </gazebo>
+        <gazebo>
+            <plugin name="joint_encoder_${name}" filename="libJointEncoder.so">
+                <joint>${name}_joint</joint>
+                <topic>/simulation/encoder/abs/${name}</topic>
+                <lower>0</lower>
+                <upper>${link_4_width/2 - finger_width}</upper>
+                <absolute>1</absolute>
+                <resolution>10000</resolution>
+            </plugin>
+        </gazebo>
+        <gazebo>
             <plugin name="joint_controller${name}" filename="libControllerPID.so">
                 <joint>${name}_joint</joint>
                 <topic>/simulation/controller/vel/${name}</topic>
-                <Kp>10</Kp>
-                <Ki>0</Ki>
+                <Kp>20</Kp>
+                <Ki>2</Ki>
                 <Kd>5</Kd>
             </plugin>

File: phobos_simulation/xacro/arm/link_0.xacro (robot description, xacro)
@@ -82,5 +82,5 @@
                 <upper>3</upper>
                 <absolute>1</absolute>
-                <resolution>3600</resolution>
+                <resolution>10000</resolution>
             </plugin>
         </gazebo>

File: phobos_simulation/xacro/arm/link_1.xacro (robot description, xacro)
@@ -79,5 +79,5 @@
                 <upper>1.6</upper>
                 <absolute>1</absolute>
-                <resolution>3600</resolution>
+                <resolution>10000</resolution>
             </plugin>
         </gazebo>

File: phobos_simulation/xacro/arm/link_2.xacro (robot description, xacro)
@@ -79,5 +79,5 @@
                 <upper>3.65</upper>
                 <absolute>1</absolute>
-                <resolution>3600</resolution>
+                <resolution>10000</resolution>
             </plugin>
         </gazebo>

File: phobos_simulation/xacro/arm/link_3.xacro (robot description, xacro)
@@ -66,5 +66,5 @@
                 <upper>1.1</upper>
                 <absolute>1</absolute>
-                <resolution>3600</resolution>
+                <resolution>10000</resolution>
             </plugin>
         </gazebo>

File: phobos_simulation/xacro/arm/link_4.xacro (robot description, xacro)
@@ -66,5 +66,5 @@
                 <upper>3.14</upper>
                 <absolute>1</absolute>
-                <resolution>3600</resolution>
+                <resolution>10000</resolution>
             </plugin>
         </gazebo>

File: phobos_simulation/xacro/rocker-bogie/bogie/bogie_bearing.xacro (robot description, xacro)
@@ -50,4 +50,14 @@
                 <dynamics damping="1"/>
             </joint>
+            <gazebo>
+                <plugin name="joint_encoder_${name}" filename="libJointEncoder.so">
+                    <joint>${name}_joint</joint>
+                    <topic>/simulation/encoder/abs/${name}</topic>
+                    <lower>-0.5</lower>
+                    <upper>0.5</upper>
+                    <absolute>1</absolute>
+                    <resolution>10000</resolution>
+                </plugin>
+            </gazebo>
             <gazebo reference="${name}_joint">
                 <provideFeedback value="true"/>

File: phobos_simulation/xacro/rocker-bogie/rocker/rocker_bearing.xacro (robot description, xacro)
@@ -50,4 +50,14 @@
                 <dynamics damping="2" friction="0"/>
             </joint>
+            <gazebo>
+                <plugin name="joint_encoder_${name}" filename="libJointEncoder.so">
+                    <joint>${name}_joint</joint>
+                    <topic>/simulation/encoder/abs/${name}</topic>
+                    <lower>-0.5</lower>
+                    <upper>0.5</upper>
+                    <absolute>1</absolute>
+                    <resolution>10000</resolution>
+                </plugin>
+            </gazebo>
             <gazebo reference="${name}_joint">
                 <provideFeedback value="true"/>

File: phobos_simulation/xacro/sensors/camera.xacro (robot description, xacro)
@@ -60,5 +60,5 @@
                     <imageTopicName>image_raw</imageTopicName>
                     <cameraInfoTopicName>camera_info</cameraInfoTopicName>
-                    <frameName>${name}_lens</frameName>
+                    <frameName>/${name}_lens</frameName>
                     <hackBaseline>0.07</hackBaseline>
                     <distortionK1>0.0</distortionK1>

Commit message: MESHES for manipulators link 0,1,2

File: phobos_simulation/xacro/arm/__arm.xacro (robot description, xacro)
@@ -17,5 +17,5 @@
     <xacro:property name="link_0_length2" value=".100"/>
     <xacro:property name="link_0_radius2" value=".070"/>
-    <xacro:property name="link_1_length" value=".500"/>
+    <xacro:property name="link_1_length" value=".452"/>
     <xacro:property name="link_1_width" value=".070"/>
     <xacro:property name="link_1_height" value=".070"/>
@@ -34,15 +34,15 @@
 <!-- LINKS -->
     <xacro:link_0 name="link_0" parent="main_body" x="${manipulator_pose_x}"            y="0"    z="${manipulator_pose_z}"/>
-    <xacro:link_1 name="link_1" parent="link_0"    x="0"              y="0"    z="${link_0_length1/2 + link_1_height/2}"/>
-    <xacro:link_2 name="link_2" parent="link_1"    x="${-link_1_length}"    y="0"    z="${link_1_height/2}"/>
-    <xacro:link_3 name="link_3" parent="link_2"    x="${link_2_length}"     y="0"    z="${link_2_height/2}"/>
-    <xacro:link_4 name="link_4" parent="link_3"    x="${link_3_length}"     y="0"    z="0"/>
+    <xacro:link_1 name="link_1" parent="link_0"    x="-0.003"              y="0"    z="${link_0_length1/2 + link_1_height/2 + 0.04}"/>
+    <xacro:link_2 name="link_2" parent="link_1"    x="${-link_1_length}"    y="0"    z="0"/>
+    <!-- <xacro:link_3 name="link_3" parent="link_2"    x="${link_2_length}"     y="0"    z="${link_2_height/2}"/> -->
+    <!-- <xacro:link_4 name="link_4" parent="link_3"    x="${link_3_length}"     y="0"    z="0"/> -->
 <!-- GRABBER -->
-    <xacro:finger name="finger_l" parent="link_4" x="${link_4_length + finger_length/2}" y="${link_4_width/2 - finger_width/2-.001}" z="${finger_height+.001}" side="-1"/>
-    <xacro:finger_b name="finger_lb" parent="finger_l" x="0" y="0" z="${-2*finger_height-.001}" side="-1"/>
-    <xacro:finger name="finger_r" parent="link_4" x="${link_4_length + finger_length/2}" y="${-link_4_width/2 + finger_width/2}" z="0" side="1"/>
-    <xacro:finger_b name="finger_rc" parent="finger_r" x="0" y="0" z="${2*finger_height+.002}" side="1"/>
-    <xacro:finger_b name="finger_rb" parent="finger_r" x="0" y="0" z="${-2*finger_height-.002}" side="1"/>
+    <!-- <xacro:finger name="finger_l" parent="link_4" x="${link_4_length + finger_length/2}" y="${link_4_width/2 - finger_width/2-.001}" z="${finger_height+.001}" side="-1"/> -->
+    <!-- <xacro:finger_b name="finger_lb" parent="finger_l" x="0" y="0" z="${-2*finger_height-.001}" side="-1"/> -->
+    <!-- <xacro:finger name="finger_r" parent="link_4" x="${link_4_length + finger_length/2}" y="${-link_4_width/2 + finger_width/2}" z="0" side="1"/> -->
+    <!-- <xacro:finger_b name="finger_rc" parent="finger_r" x="0" y="0" z="${2*finger_height+.002}" side="1"/> -->
+    <!-- <xacro:finger_b name="finger_rb" parent="finger_r" x="0" y="0" z="${-2*finger_height-.002}" side="1"/> -->
 <!-- SENSORS -->
-    <xacro:camera_link name="camera4" parent="link_4" x=".030" y="0" z=".100" pitch="0.4"/>
+    <!-- <xacro:camera_link name="camera4" parent="link_4" x=".030" y="0" z=".100" pitch="0.4"/> -->
 </robot>

File: phobos_simulation/xacro/arm/link_0.xacro (robot description, xacro)
@@ -15,4 +15,11 @@
         </geometry>
     </xacro:macro>
+<!-- VISUAL -->
+    <xacro:macro name="link_0_visual">
+        <origin xyz="0.085 0.112 -0.01" rpy="1.57075 0 -1.448"/>
+        <geometry>
+            <mesh filename="package://phobos_meshes/rover_stl/stopien_2.STL" scale="0.001 0.001 0.001"/>
+        </geometry>
+    </xacro:macro>
 <!-- MATERIAL -->
     <xacro:macro name="link_0_material">
@@ -26,9 +33,5 @@
         <link name="${name}">
             <visual>
-                <xacro:link_0_geometry1/>
-                <xacro:link_0_material/>
-            </visual>
-            <visual>
-                <xacro:link_0_geometry2/>
+                <xacro:link_0_visual/>
                 <xacro:link_0_material/>
             </visual>

File: phobos_simulation/xacro/arm/link_1.xacro (robot description, xacro)
@@ -14,4 +14,11 @@
         </geometry>
     </xacro:macro>
+<!-- VISUAL -->
+    <xacro:macro name="link_1_visual">
+        <origin xyz="0.07 -0.05 -0.050" rpy="0.045 0.13 1.57075"/>
+        <geometry>
+            <mesh filename="package://phobos_meshes/rover_stl/stopien_3.STL" scale="0.001 0.001 0.001"/>
+        </geometry>
+    </xacro:macro>
 <!-- MATERIAL -->
     <xacro:macro name="link_1_material">
@@ -24,9 +31,5 @@
         <link name="${name}">
             <visual>
-                <xacro:link_1_geometry_1/>
-                <xacro:link_1_material/>
-            </visual>
-            <visual>
-                <xacro:link_1_geometry_2/>
+                <xacro:link_1_visual/>
                 <xacro:link_1_material/>
             </visual>

File: phobos_simulation/xacro/arm/link_2.xacro (robot description, xacro)
@@ -14,4 +14,11 @@
         </geometry>
     </xacro:macro>
+    <!-- VISUAL -->
+    <xacro:macro name="link_2_visual">
+        <origin xyz="0.34 0.093 -0.523" rpy="1.57075 0 -1.45"/>
+        <geometry>
+            <mesh filename="package://phobos_meshes/rover_stl/stopien_4.STL" scale="0.001 0.001 0.001"/>
+        </geometry>
+    </xacro:macro>
 <!-- MATERIAL -->
     <xacro:macro name="link_2_material">
@@ -24,9 +31,5 @@
         <link name="${name}">
             <visual>
-                <xacro:link_2_geometry_1/>
-                <xacro:link_2_material/>
-            </visual>
-            <visual>
-                <xacro:link_2_geometry_2/>
+                <xacro:link_2_visual/>
                 <xacro:link_2_material/>
             </visual>

File: phobos_simulation/xacro/arm/link_3.xacro (robot description, xacro)
@@ -14,9 +14,16 @@
         </material>
     </xacro:macro>
+    <!-- VISUAL -->
+    <xacro:macro name="link_3_visual">
+        <origin xyz="0 0 0" rpy="0 0 0"/>
+        <geometry>
+            <mesh filename="package://phobos_meshes/rover_stl/stopien_5.STL" scale="0.001 0.001 0.001"/>
+        </geometry>
+    </xacro:macro>
 <!-- LINK -->
     <xacro:macro name="link_3" params="name parent x y z">
         <link name="${name}">
             <visual>
-                <xacro:link_3_geometry/>
+                <xacro:link_3_visual/>
                 <xacro:link_3_material/>
             </visual>

File: phobos_simulation/xacro/arm/link_4.xacro (robot description, xacro)
@@ -6,4 +6,11 @@
         <geometry>
             <box size="${link_4_length} ${link_4_width} ${link_4_height}"/>
+        </geometry>
+    </xacro:macro>
+    <!-- VISUAL -->
+    <xacro:macro name="link_4_visual">
+        <origin xyz="0 0 0" rpy="0 0 0"/>
+        <geometry>
+            <mesh filename="package://phobos_meshes/rover_stl/chwytak.STL" scale="0.001 0.001 0.001"/>
         </geometry>
     </xacro:macro>
@@ -18,5 +25,5 @@
         <link name="${name}">
             <visual>
-                <xacro:link_4_geometry/>
+                <xacro:link_4_visual/>
                 <xacro:link_4_material/>
             </visual>

File: phobos_simulation/xacro/base/main_body.xacro (robot description, xacro)
@@ -33,8 +33,14 @@
     </xacro:macro> -->
 <!-- VISUAL -->
-    <xacro:macro name="main_body_visual">
+    <xacro:macro name="main_body_visual_1">
         <origin xyz="-0.402 0.43 -0.294" rpy="1.57075 0 0"/>
         <geometry>
             <mesh filename="package://phobos_meshes/rover_stl/R.Assembly.STL" scale="0.001 0.001 0.001"/>
+        </geometry>
+    </xacro:macro>
+    <xacro:macro name="main_body_visual_2">
+        <origin xyz="0.036 -0.165 -0.0735" rpy="1.57075 0 1.88"/>
+        <geometry>
+            <mesh filename="package://phobos_meshes/rover_stl/podstawa_manipulatora.STL" scale="0.001 0.001 0.001"/>
         </geometry>
     </xacro:macro>
@@ -50,5 +56,9 @@
         <link name="${name}">
             <visual>
-                <xacro:main_body_visual/>
+                <xacro:main_body_visual_1/>
+                <xacro:main_body_material/>
+            </visual>
+            <visual>
+                <xacro:main_body_visual_2/>
                 <xacro:main_body_material/>
             </visual>

Commit message: MESHES for manipulators link 0,1,2,3

File: phobos_simulation/xacro/arm/__arm.xacro (robot description, xacro)
@@ -20,8 +20,8 @@
     <xacro:property name="link_1_width" value=".070"/>
     <xacro:property name="link_1_height" value=".070"/>
-    <xacro:property name="link_2_length" value=".250"/>
+    <xacro:property name="link_2_length" value=".308"/>
     <xacro:property name="link_2_width" value=".050"/>
     <xacro:property name="link_2_height" value=".050"/>
-    <xacro:property name="link_3_length" value=".250"/>
+    <xacro:property name="link_3_length" value=".090"/>
     <xacro:property name="link_3_width" value=".040"/>
     <xacro:property name="link_3_height" value=".040"/>
@@ -36,6 +36,6 @@
     <xacro:link_1 name="link_1" parent="link_0"    x="-0.003"              y="0"    z="${link_0_length1/2 + link_1_height/2 + 0.04}"/>
     <xacro:link_2 name="link_2" parent="link_1"    x="${-link_1_length}"    y="0"    z="0"/>
-    <!-- <xacro:link_3 name="link_3" parent="link_2"    x="${link_2_length}"     y="0"    z="${link_2_height/2}"/> -->
-    <!-- <xacro:link_4 name="link_4" parent="link_3"    x="${link_3_length}"     y="0"    z="0"/> -->
+    <xacro:link_3 name="link_3" parent="link_2"    x="${link_2_length}"     y="0"    z="${link_2_height/2 + 0.025}"/>
+    <xacro:link_4 name="link_4" parent="link_3"    x="${link_3_length}"     y="0"    z="0"/>
 <!-- GRABBER -->
     <!-- <xacro:finger name="finger_l" parent="link_4" x="${link_4_length + finger_length/2}" y="${link_4_width/2 - finger_width/2-.001}" z="${finger_height+.001}" side="-1"/> -->

File: phobos_simulation/xacro/arm/link_1.xacro (robot description, xacro)
@@ -16,5 +16,5 @@
 <!-- VISUAL -->
     <xacro:macro name="link_1_visual">
-        <origin xyz="0.07 -0.05 -0.050" rpy="0.045 0.13 1.57075"/>
+        <origin xyz="0.07 -0.055 -0.050" rpy="0.045 0.13 1.57075"/>
         <geometry>
             <mesh filename="package://phobos_meshes/rover_stl/stopien_3.STL" scale="0.001 0.001 0.001"/>

File: phobos_simulation/xacro/arm/link_2.xacro (robot description, xacro)
@@ -16,5 +16,5 @@
     <!-- VISUAL -->
     <xacro:macro name="link_2_visual">
-        <origin xyz="0.34 0.093 -0.523" rpy="1.57075 0 -1.45"/>
+        <origin xyz="0.34 0.088 -0.523" rpy="1.57075 0 -1.45"/>
         <geometry>
             <mesh filename="package://phobos_meshes/rover_stl/stopien_4.STL" scale="0.001 0.001 0.001"/>

File: phobos_simulation/xacro/arm/link_3.xacro (robot description, xacro)
@@ -16,5 +16,5 @@
     <!-- VISUAL -->
     <xacro:macro name="link_3_visual">
-        <origin xyz="0 0 0" rpy="0 0 0"/>
+        <origin xyz="0.112 -0.051 0.568" rpy="-1.52 0 1.45"/>
         <geometry>
             <mesh filename="package://phobos_meshes/rover_stl/stopien_5.STL" scale="0.001 0.001 0.001"/>

File: phobos_simulation/xacro/arm/link_4.xacro (robot description, xacro)
@@ -10,5 +10,5 @@
     <!-- VISUAL -->
     <xacro:macro name="link_4_visual">
-        <origin xyz="0 0 0" rpy="0 0 0"/>
+        <origin xyz="0 0 0" rpy="0.1 0 0"/>
         <geometry>
             <mesh filename="package://phobos_meshes/rover_stl/chwytak.STL" scale="0.001 0.001 0.001"/>

Commit message: link 4 moved

File: phobos_simulation/xacro/arm/__arm.xacro (robot description, xacro)
@@ -8,5 +8,4 @@
     <xacro:include filename="link_4.xacro"/>
     <xacro:include filename="finger.xacro"/>
-    <xacro:include filename="finger_b.xacro"/>
     <xacro:include filename="../sensors/camera.xacro"/>
 <!-- PROPERTIES -->
@@ -29,7 +28,7 @@
     <xacro:property name="link_4_width" value=".200"/>
     <xacro:property name="link_4_height" value=".152"/>
-    <xacro:property name="finger_length" value=".130"/>
+    <xacro:property name="finger_length" value=".250"/>
     <xacro:property name="finger_width" value=".010"/>
-    <xacro:property name="finger_height" value=".030"/>
+    <xacro:property name="finger_height" value=".070"/>
 <!-- LINKS -->
     <xacro:link_0 name="link_0" parent="main_body" x="${manipulator_pose_x}"            y="0"    z="${manipulator_pose_z}"/>
@@ -37,5 +36,6 @@
     <xacro:link_2 name="link_2" parent="link_1"    x="${-link_1_length}"    y="0"    z="0"/>
     <xacro:link_3 name="link_3" parent="link_2"    x="${link_2_length}"     y="0"    z="${link_2_height/2 + 0.025}"/>
-    <xacro:link_4 name="link_4" parent="link_3"    x="${link_3_length}"     y="0"    z="0"/>
+    <xacro:link_4 name="link_4" parent="link_3"    x="${link_3_length}"     y="0.002"    z="0"/>
+    <!-- <xacro:finger name="finger" parent="link_4"    x=".073"     y="0.04"    z="0" side="-1"/> -->
 <!-- GRABBER -->
     <!-- <xacro:finger name="finger_l" parent="link_4" x="${link_4_length + finger_length/2}" y="${link_4_width/2 - finger_width/2-.001}" z="${finger_height+.001}" side="-1"/> -->

File: phobos_simulation/xacro/arm/link_4.xacro (robot description, xacro)
@@ -10,5 +10,7 @@
     <!-- VISUAL -->
     <xacro:macro name="link_4_visual">
-        <origin xyz="0.25 0.1 -0.587" rpy="1.57075 -0.15 -1.45"/>
+        <!-- <origin xyz="0.25 0.1 -0.587" rpy="1.8 -0.5 -1.45"/> -->
+        <!-- <origin xyz="0.25 0.1 -0.587" rpy="1.57075 -0.1 -1.45"/> -->
+        <origin xyz="0.265 0.0835 -0.583" rpy="1.59 -0.18 -1.45"/>
         <geometry>
             <mesh filename="package://phobos_meshes/rover_stl/chwytak.STL" scale="0.001 0.001 0.001"/>
