Commit message: All MESHES added, proper collisions for gripper

File: phobos_simulation/xacro/arm/__arm.xacro (robot description, xacro)
@@ -7,4 +7,5 @@
     <xacro:include filename="link_3.xacro"/>
     <xacro:include filename="link_4.xacro"/>
+    <xacro:include filename="link_4_finger.xacro"/>
     <xacro:include filename="finger.xacro"/>
     <xacro:include filename="../sensors/camera.xacro"/>
@@ -26,9 +27,12 @@
     <xacro:property name="link_3_height" value=".040"/>
     <xacro:property name="link_4_length" value=".050"/>
-    <xacro:property name="link_4_width" value=".200"/>
-    <xacro:property name="link_4_height" value=".152"/>
-    <xacro:property name="finger_length" value=".250"/>
-    <xacro:property name="finger_width" value=".010"/>
+    <xacro:property name="link_4_width" value=".100"/>
+    <xacro:property name="link_4_height" value=".100"/>
+    <xacro:property name="finger_length" value=".350"/>
+    <xacro:property name="finger_width" value=".003"/>
     <xacro:property name="finger_height" value=".070"/>
+    <xacro:property name="link_4_finger_length" value=".350"/>
+    <xacro:property name="link_4_finger_width" value=".003"/>
+    <xacro:property name="link_4_finger_height" value=".070"/>
 <!-- LINKS -->
     <xacro:link_0 name="link_0" parent="main_body" x="${manipulator_pose_x}"            y="0"    z="${manipulator_pose_z}"/>
@@ -37,5 +41,6 @@
     <xacro:link_3 name="link_3" parent="link_2"    x="${link_2_length}"     y="0"    z="${link_2_height/2 + 0.025}"/>
     <xacro:link_4 name="link_4" parent="link_3"    x="${link_3_length}"     y="0.002"    z="0"/>
-    <!-- <xacro:finger name="finger" parent="link_4"    x=".073"     y="0.04"    z="0" side="-1"/> -->
+    <xacro:finger name="finger" parent="link_4"    x=".073"     y="0.04"    z="0" side="-1"/>
+    <xacro:link_4_finger name="link_4_finger" parent="link_4"    x=".073"     y="-0.04"    z="0" side="1"/>
 <!-- GRABBER -->
     <!-- <xacro:finger name="finger_l" parent="link_4" x="${link_4_length + finger_length/2}" y="${link_4_width/2 - finger_width/2-.001}" z="${finger_height+.001}" side="-1"/> -->

File: phobos_simulation/xacro/arm/link_2.xacro (robot description, xacro)
@@ -3,5 +3,5 @@
 <!-- GEOMETRY -->
     <xacro:macro name="link_2_geometry_1">
-        <origin rpy="0 0 0" xyz="${link_2_length/2} 0 ${link_2_height/2}" />
+        <origin rpy="0 0 0" xyz="${link_2_length/2} 0 ${link_2_height/2 + 0.06}" />
         <geometry>
             <box size="${link_2_length} ${link_2_width} ${link_2_height}"/>

File: phobos_simulation/xacro/arm/link_4.xacro (robot description, xacro)
@@ -1,4 +1,5 @@
 <?xml version="1.0"?>
 <robot xmlns:xacro="http://www.ros.org/wiki/xacro" name="link_4">
+<xacro:include filename="finger.xacro"/>
 <!-- GEOMETRY -->
     <xacro:macro name="link_4_geometry">
@@ -10,6 +11,4 @@
     <!-- VISUAL -->
     <xacro:macro name="link_4_visual">
-        <!-- <origin xyz="0.25 0.1 -0.587" rpy="1.8 -0.5 -1.45"/> -->
-        <!-- <origin xyz="0.25 0.1 -0.587" rpy="1.57075 -0.1 -1.45"/> -->
         <origin xyz="0.265 0.0835 -0.583" rpy="1.59 -0.18 -1.45"/>
         <geometry>

File: phobos_simulation/xacro/arm/link_4_finger.xacro (robot description, xacro)
@@ -1,43 +1,43 @@
 <?xml version="1.0"?>
-<robot xmlns:xacro="http://www.ros.org/wiki/xacro" name="finger">
+<robot xmlns:xacro="http://www.ros.org/wiki/xacro" name="link_4_finger">
 <!-- GEOMETRY -->
-    <xacro:macro name="finger_geometry_1">
-        <origin rpy="0 0 0" xyz="${finger_length/4} 0 0" />
+    <xacro:macro name="link_4_finger_geometry_1">
+        <origin rpy="0 0 0" xyz="${link_4_finger_length/4} 0 0" />
         <geometry>
-            <box size="${finger_length/2} ${finger_width} ${finger_height}"/>
+            <box size="${link_4_finger_length/2} ${link_4_finger_width} ${link_4_finger_height}"/>
         </geometry>
     </xacro:macro>
-    <xacro:macro name="finger_geometry_2">
-        <origin rpy="0 0 ${1*side}" xyz="${finger_length/2 + 0.007} ${0.013*side} 0" />
+    <xacro:macro name="link_4_finger_geometry_2">
+        <origin rpy="0 0 ${1*side}" xyz="${link_4_finger_length/2 + 0.007} ${0.013*side} 0" />
         <geometry>
-            <box size="0.033 ${finger_width} ${finger_height}"/>
+            <box size="0.033 ${link_4_finger_width} ${link_4_finger_height}"/>
         </geometry>
     </xacro:macro>
-    <xacro:macro name="finger_geometry_3">
-        <origin rpy="1.57075 0 0" xyz="${finger_length/2-0.01} ${side*0.027} ${finger_height/2}" />
+    <xacro:macro name="link_4_finger_geometry_3">
+        <origin rpy="1.57075 0 0" xyz="${link_4_finger_length/2-0.01} ${side*0.027} ${link_4_finger_height/2}" />
         <geometry>
             <box size="0.05 0.003 0.003"/>
         </geometry>
     </xacro:macro>
-    <xacro:macro name="finger_geometry_4">
-        <origin rpy="1.57075 0 0" xyz="${finger_length/2-0.01} ${side*0.027} ${-finger_height/2}" />
+    <xacro:macro name="link_4_finger_geometry_4">
+        <origin rpy="1.57075 0 0" xyz="${link_4_finger_length/2-0.01} ${side*0.027} ${-link_4_finger_height/2}" />
         <geometry>
             <box size="0.05 0.003 0.003"/>
         </geometry>
     </xacro:macro>
-    <!-- <xacro:macro name="finger_geometry_3">
-        <origin rpy="0 0 ${1*side}" xyz="${finger_length/2} 0 0" />
+    <!-- <xacro:macro name="link_4_finger_geometry_3">
+        <origin rpy="0 0 ${1*side}" xyz="${link_4_finger_length/2} 0 0" />
         <geometry>
-            <cylinder length="${finger_height}" radius="${finger_width/2}"/>
+            <cylinder length="${link_4_finger_height}" radius="${link_4_finger_width/2}"/>
         </geometry>
     </xacro:macro>
-    <xacro:macro name="finger_geometry_4">
-        <origin rpy="0 0 ${1*side}" xyz="${finger_length/2+finger_length/6*1.414} ${finger_length/6*1.414*side} 0" />
+    <xacro:macro name="link_4_finger_geometry_4">
+        <origin rpy="0 0 ${1*side}" xyz="${link_4_finger_length/2+link_4_finger_length/6*1.414} ${link_4_finger_length/6*1.414*side} 0" />
         <geometry>
-            <cylinder length="${finger_height}" radius="${finger_width/2}"/>
+            <cylinder length="${link_4_finger_height}" radius="${link_4_finger_width/2}"/>
         </geometry>
     </xacro:macro> -->
 <!-- VISUAL -->
-    <xacro:macro name="finger_visual">
+    <xacro:macro name="link_4_finger_visual">
         <origin xyz="0.195 -0.078 -0.571" rpy="1.59 -0.18 -1.75"/>
         <geometry>
@@ -46,43 +46,43 @@
     </xacro:macro>
 <!-- MATERIAL -->
-    <xacro:macro name="finger_material">
-        <material name="finger_color">
+    <xacro:macro name="link_4_finger_material">
+        <material name="link_4_finger_color">
             <color rgba=".4 .4 .8 1"/>
         </material>
     </xacro:macro>
 <!-- LINK -->
-    <xacro:macro name="finger" params="name parent x y z side">
+    <xacro:macro name="link_4_finger" params="name parent x y z side">
         <link name="${name}">
-            <visual>
-                <xacro:finger_visual/>
-                <xacro:finger_material/>
-            </visual>
             <!-- <visual>
-                <xacro:finger_geometry_1/>
-                <xacro:finger_material/>
+                <xacro:link_4_finger_visual/>
+                <xacro:link_4_finger_material/>
+            </visual> -->
+            <!-- <visual>
+                <xacro:link_4_finger_geometry_1/>
+                <xacro:link_4_finger_material/>
             </visual>
             <visual>
-                <xacro:finger_geometry_2/>
-                <xacro:finger_material/>
+                <xacro:link_4_finger_geometry_2/>
+                <xacro:link_4_finger_material/>
             </visual>
             <visual>
-                <xacro:finger_geometry_3/>
-                <xacro:finger_material/>
+                <xacro:link_4_finger_geometry_3/>
+                <xacro:link_4_finger_material/>
             </visual>
             <visual>
-                <xacro:finger_geometry_4/>
-                <xacro:finger_material/>
+                <xacro:link_4_finger_geometry_4/>
+                <xacro:link_4_finger_material/>
             </visual> -->
             <collision>
-                <xacro:finger_geometry_1/>
+                <xacro:link_4_finger_geometry_1/>
             </collision>
             <collision>
-                <xacro:finger_geometry_2/>
+                <xacro:link_4_finger_geometry_2/>
             </collision>
             <collision>
-                <xacro:finger_geometry_3/>
+                <xacro:link_4_finger_geometry_3/>
             </collision>
             <collision>
-                <xacro:finger_geometry_4/>
+                <xacro:link_4_finger_geometry_4/>
             </collision>
             <inertial>
@@ -98,11 +98,8 @@
             <selfCollide>True</selfCollide>
         </gazebo>
-        <joint name="${name}_joint" type="revolute">
+        <joint name="${name}_joint" type="fixed">
             <parent link="${parent}"/>
             <child link="${name}"/>
             <origin rpy="0 0 0" xyz="${x} ${y} ${z}"/>
-            <axis xyz="0 0 1"/>
-            <limit effort="10000" velocity="1" lower="-0.12" upper="0.45"/>
-            <dynamics damping=".1"/>
         </joint>
         <!--gazebo reference="${name}_joint">
@@ -113,10 +110,10 @@
             <fudgeFactor>0.0</fudgeFactor>
         </gazebo-->
-        <gazebo>
+        <!-- <gazebo>
             <plugin name="joint_limiter_${name}" filename="libJointLimiter.so">
                 <joint>${name}_joint</joint>
                 <topic>/simulation/controller/vel/${name}</topic>
                 <lower>0</lower>
-                <upper>${link_4_width/2 - finger_width}</upper>
+                <upper>${link_4_width/2 - link_4_finger_width}</upper>
             </plugin>
         </gazebo>
@@ -126,5 +123,5 @@
                 <topic>/simulation/encoder/abs/${name}</topic>
                 <lower>0</lower>
-                <upper>${link_4_width/2 - finger_width}</upper>
+                <upper>${link_4_width/2 - link_4_finger_width}</upper>
                 <absolute>1</absolute>
                 <resolution>10000</resolution>
@@ -136,5 +133,5 @@
                 <topic>/simulation/encoder/abs/${name}</topic>
                 <lower>0</lower>
-                <upper>${link_4_width/2 - finger_width}</upper>
+                <upper>${link_4_width/2 - link_4_finger_width}</upper>
                 <absolute>1</absolute>
                 <resolution>10000</resolution>
@@ -149,5 +146,5 @@
                 <Kd>5</Kd>
             </plugin>
-        </gazebo>
+        </gazebo> -->
         <!--transmission name="${name}_transmission">
             <type>transmission_interface/SimpleTransmission</type>
