Commit message: plugins topics changed

File: phobos_simulation/xacro/sensors/camera.xacro (robot description, xacro)
@@ -32,5 +32,5 @@
     </xacro:macro>
 <!-- CAMERA GAZEBO PLUGIN -->
-    <xacro:macro name="camera_plugin" params="name width height">
+    <xacro:macro name="camera_plugin" params="name">
         <gazebo reference="${name}">
             <sensor type="camera" name="${name}">
@@ -40,6 +40,6 @@
                     <horizontal_fov>2</horizontal_fov>
                     <image>
-                        <width>${width}</width>
-                        <height>${height}</height>
+                        <width>320</width>
+                        <height>240</height>
                         <format>B8G8R8</format>
                     </image>
@@ -123,5 +123,5 @@
             <selfCollide> false </selfCollide>
         </gazebo>
-        <xacro:camera_plugin name="${name}" width="320" height="240"/>
+        <xacro:camera_plugin name="${name}"/>
     </xacro:macro>
 </robot>
