Commit message: MESHES for frame and suspension added to .urdf model

File: phobos_simulation/xacro/base/main_body.xacro (robot description, xacro)
@@ -32,4 +32,11 @@
         </geometry>
     </xacro:macro> -->
+<!-- VISUAL -->
+    <xacro:macro name="main_body_visual">
+        <origin xyz="-0.402 0.43 -0.294" rpy="1.57075 0 0"/>
+        <geometry>
+            <mesh filename="package://phobos_meshes/rover_stl/R.Assembly.STL" scale="0.001 0.001 0.001"/>
+        </geometry>
+    </xacro:macro>
 <!-- MATERIAL -->
     <xacro:macro name="main_body_material">
@@ -43,5 +50,5 @@
         <link name="${name}">
             <visual>
-                <xacro:main_body_geometry_1/>
+                <xacro:main_body_visual/>
                 <xacro:main_body_material/>
             </visual>

File: phobos_simulation/xacro/rocker-bogie/bogie/bogie_bearing.xacro (robot description, xacro)
@@ -6,4 +6,17 @@
         <geometry>
             <cylinder length="${bogie_bearing_length}" radius="${bogie_bearing_radius}"/>
+        </geometry>
+    </xacro:macro>
+<!-- VISUAL -->
+    <xacro:macro name="bogie_visual_left">
+        <origin xyz="-0.288 -.230 -0.21" rpy="1.57075 0 1.57075"/>
+        <geometry>
+            <mesh filename="package://phobos_meshes/rover_stl/bogie_lewe_stl.STL" scale="0.001 0.001 0.001"/>
+        </geometry>
+    </xacro:macro>
+    <xacro:macro name="bogie_visual_right">
+        <origin xyz="-0.288 -.195 -0.21" rpy="1.57075 0 1.57075"/>
+        <geometry>
+            <mesh filename="package://phobos_meshes/rover_stl/bogie_prawe_stl.STL" scale="0.001 0.001 0.001"/>
         </geometry>
     </xacro:macro>
@@ -18,6 +31,7 @@
         <link name="${name}">
             <visual>
-                <xacro:bogie_bearing_geometry/>
-                <xacro:bogie_bearing_material/>
+                <xacro:if value="${side == 1}"> <xacro:bogie_visual_left/> </xacro:if>
+                <xacro:if value="${side == -1}"> <xacro:bogie_visual_right/> </xacro:if>
+                <xacro:rocker_material/>
             </visual>
             <collision>

File: phobos_simulation/xacro/rocker-bogie/rocker/rocker_bearing.xacro (robot description, xacro)
@@ -6,4 +6,17 @@
         <geometry>
             <cylinder length="${rocker_bearing_length}" radius="${rocker_bearing_radius}"/>
+        </geometry>
+    </xacro:macro>
+<!-- VISUAL -->
+    <xacro:macro name="rocker_visual_left">
+        <origin xyz="-0.14 -.775 -0.16" rpy="1.57075 0 3.1416"/>
+        <geometry>
+            <mesh filename="package://phobos_meshes/rover_stl/rocker_lewy_stl.STL" scale="0.001 0.001 0.001"/>
+        </geometry>
+    </xacro:macro>
+    <xacro:macro name="rocker_visual_right">
+        <origin xyz="-0.14 -.739 -0.16" rpy="1.57075 0 3.1416"/>
+        <geometry>
+            <mesh filename="package://phobos_meshes/rover_stl/rocker_prawy_stl.STL" scale="0.001 0.001 0.001"/>
         </geometry>
     </xacro:macro>
@@ -18,5 +31,6 @@
         <link name="${name}">
             <visual>
-                <xacro:rocker_geometry/>
+                <xacro:if value="${side == 1}"> <xacro:rocker_visual_left/> </xacro:if>
+                <xacro:if value="${side == -1}"> <xacro:rocker_visual_right/> </xacro:if>
                 <xacro:rocker_material/>
             </visual>

File: phobos_simulation/xacro/rocker-bogie/wheel.xacro (robot description, xacro)
@@ -6,4 +6,11 @@
         <geometry>
             <cylinder length="${wheel_width}" radius="${wheel_radius}"/>
+        </geometry>
+    </xacro:macro>
+<!-- VISUAL -->
+    <xacro:macro name="wheel_visual">
+        <origin xyz="0.01 -0.05 -0.13" rpy="0 0 1.57075"/>
+        <geometry>
+            <mesh filename="package://phobos_meshes/rover_stl/kolo_stl.STL" scale="0.001 0.001 0.001"/>
         </geometry>
     </xacro:macro>
@@ -18,5 +25,5 @@
         <link name="wheel_${name}">
             <visual>
-                <xacro:wheel_geometry/>
+                <xacro:wheel_visual/>
                 <xacro:wheel_material/>
             </visual>
